Commit message: Initial commit from semestral project

File: myGym/envs/robots/real_hands/humanoid_with_hands.urdf (robot description, URDF)
Before this commit: robot , 89 links, 88 joints
Links:
- removed link l_l_arm
- removed link l_l_forearm
- removed link l_l_index0
- removed link l_l_index1
- removed link l_l_index2
- removed link l_l_index3
- removed link l_l_middle0
- removed link l_l_middle1
- removed link l_l_middle2
- removed link l_l_middle3
- removed link l_l_palm
- removed link l_l_pinky0
- removed link l_l_pinky1
- removed link l_l_pinky2
- removed link l_l_pinky3
- removed link l_l_ring0
- removed link l_l_ring1
- removed link l_l_ring2
- removed link l_l_ring3
- removed link l_l_thumb0
- removed link l_l_thumb1
- removed link l_l_thumb2
- removed link l_l_thumb3
- removed link l_l_wristx
- removed link l_l_wristy
- removed link l_l_wristz
- removed link l_link0_1
- removed link l_link0_10
- removed link l_link0_12
- removed link l_link0_15
- removed link l_link0_17
- removed link l_link0_19
- removed link l_link0_2
- removed link l_link0_21
- removed link l_link0_23
- removed link l_link0_25
- removed link l_link0_27
- removed link l_link0_29
- removed link l_link0_3
- removed link l_link0_32
- removed link l_link0_34
- removed link l_link0_36
- removed link l_link0_38
- removed link l_link0_40
- removed link l_link0_42
- removed link l_link0_44
- removed link l_link0_46
- removed link l_link0_48
- removed link l_link0_5
- removed link l_link0_50
- removed link l_link0_52
- removed link l_link0_6
- removed link l_link0_8
- removed link link0_1
- removed link link0_10
- removed link link0_12
- removed link link0_2
- removed link link0_23
- removed link link0_25
- removed link link0_27
- removed link link0_29
- removed link link0_3
- removed link link0_5
- removed link link0_6
- removed link link0_8
- removed link r_arm
- added link head, mass 4.0; collision sphere radius=0.11; visual sphere radius=0.11
- added link l_elbow_base
- added link l_forearm, mass 1.05512; visual capsule length=0.23 radius=0.035
- added link l_index0, mass 0.00296; visual mesh filename=mesh/left/index0_left.stl scale=1 1 1
- added link l_index1, mass 0.00478; visual mesh filename=mesh/left/index1_left.stl scale=1 1 1
- added link l_index2, mass 0.00345; visual mesh filename=mesh/left/index2_left.stl scale=1 1 1
- added link l_index3, mass 0.00274; visual mesh filename=mesh/left/index3_left.stl scale=1 1 1
- added link l_palm, mass 0.11987; visual mesh filename=mesh/left/palm_left.stl scale=1 1 1
- added link l_shoulder_base
- added link l_shoulder_lift
- added link l_upper_arm, mass 1.05512; visual capsule length=0.23 radius=0.035
- added link l_wristx, mass 0.01069; visual mesh filename=mesh/left/wristx_left.stl scale=1 1 1
- added link l_wristy, mass 0.02729; visual mesh filename=mesh/left/wristy_left.stl scale=1 1 1
- added link l_wristz, mass 0.00602; visual mesh filename=mesh/left/wristz_left.stl scale=1 1 1
- added link r_elbow_base
- added link r_shoulder_base
- added link r_shoulder_lift
- added link r_upper_arm, mass 1.05512; collision capsule length=0.23 radius=0.035; visual capsule length=0.23 radius=0.035
- link direction_cone: geometry visual mesh filename=mesh/cone.stl scale=0.003 0.003 0.006
- link ee_x_axis: geometry visual cylinder length=0.03 radius=0.002
- link ee_y_axis: geometry visual cylinder length=0.03 radius=0.002
- link ee_z_axis: geometry visual cylinder length=0.03 radius=0.002
- link gripper: geometry collision mesh filename=mesh/right/index3.stl scale=1 1 1; visual mesh filename=mesh/right/index3.stl scale=1 1 1
- link left_foot: geometry collision box size=0.15 0.08 0.03; visual box size=0.15 0.08 0.03
- link left_shin: geometry collision capsule length=0.35 radius=0.049; visual capsule length=0.35 radius=0.049
- link left_thigh: geometry collision capsule length=0.40 radius=0.06; visual capsule length=0.40 radius=0.06
- link lwaist: mass 4.55740 -> 4.5574; geometry collision capsule length=0.12 radius=0.08; visual capsule length=0.12 radius=0.08
- link pelvis: geometry collision capsule length=0.14 radius=0.10; visual capsule length=0.14 radius=0.10
- link r_forearm: geometry collision capsule length=0.23 radius=0.035; visual capsule length=0.23 radius=0.035
- link r_index0: geometry collision mesh filename=mesh/right/index0.stl scale=1 1 1; visual mesh filename=mesh/right/index0.stl scale=1 1 1
- link r_index1: geometry collision mesh filename=mesh/right/index1.stl scale=1 1 1; visual mesh filename=mesh/right/index1.stl scale=1 1 1
- link r_index2: geometry collision mesh filename=mesh/right/index2.stl scale=1 1 1; visual mesh filename=mesh/right/index2.stl scale=1 1 1
- link r_palm: geometry collision mesh filename=mesh/right/palm.stl scale=1 1 1; visual mesh filename=mesh/right/palm.stl scale=1 1 1
- link r_wristx: geometry collision mesh filename=mesh/right/wristx.stl scale=1 1 1; visual mesh filename=mesh/right/wristx.stl scale=1 1 1
- link r_wristy: geometry collision mesh filename=mesh/right/wristy.stl scale=1 1 1; visual mesh filename=mesh/right/wristy.stl scale=1 1 1
- link r_wristz: geometry collision mesh filename=mesh/right/wristz.stl scale=1 1 1; visual mesh filename=mesh/right/wristz.stl scale=1 1 1
- link right_foot: geometry collision box size=0.15 0.08 0.03; visual box size=0.15 0.08 0.03
- link right_shin: geometry collision capsule length=0.35 radius=0.049; visual capsule length=0.35 radius=0.049
- link right_thigh: geometry collision capsule length=0.40 radius=0.06; visual capsule length=0.40 radius=0.06
- link torso: geometry collision capsule length=0.12 radius=0.08; collision capsule length=0.14 radius=0.09
Joints:
- removed joint jointfix_0_4
- removed joint jointfix_1_3
- removed joint jointfix_20_11
- removed joint jointfix_21_12
- removed joint jointfix_22_10
- removed joint jointfix_23_8
- removed joint jointfix_24_6
- removed joint jointfix_25_3
- removed joint jointfix_2_2
- removed joint jointfix_3_7
- removed joint jointfix_4_29
- removed joint jointfix_4_6
- removed joint jointfix_5_2
- removed joint jointfix_5_27
- removed joint jointfix_6_1
- removed joint jointfix_6_25
- removed joint jointfix_7_0
- removed joint jointfix_7_23
- removed joint l_jointfix_0_21
- removed joint l_jointfix_10_32
- removed joint l_jointfix_11_13
- removed joint l_jointfix_12_44
- removed joint l_jointfix_13_42
- removed joint l_jointfix_14_40
- removed joint l_jointfix_15_38
- removed joint l_jointfix_16_52
- removed joint l_jointfix_17_50
- removed joint l_jointfix_18_48
- removed joint l_jointfix_19_46
- removed joint l_jointfix_1_19
- removed joint l_jointfix_20_11
- removed joint l_jointfix_21_12
- removed joint l_jointfix_22_10
- removed joint l_jointfix_23_8
- removed joint l_jointfix_24_6
- removed joint l_jointfix_25_3
- removed joint l_jointfix_2_17
- removed joint l_jointfix_3_15
- removed joint l_jointfix_4_29
- removed joint l_jointfix_5_27
- removed joint l_jointfix_6_25
- removed joint l_jointfix_7_23
- removed joint l_jointfix_8_36
- removed joint l_jointfix_9_34
- removed joint l_l_elbow
- removed joint l_l_elbow_twist
- removed joint l_l_index_ABD
- removed joint l_l_index_DIP
- removed joint l_l_index_MCP
- removed joint l_l_index_PIP
- removed joint l_l_middle_DIP
- removed joint l_l_middle_MCP
- removed joint l_l_middle_PIP
- removed joint l_l_pinky_ABD
- removed joint l_l_pinky_DIP
- removed joint l_l_pinky_MCP
- removed joint l_l_pinky_PIP
- removed joint l_l_ring_ABD
- removed joint l_l_ring_DIP
- removed joint l_l_ring_MCP
- removed joint l_l_ring_PIP
- removed joint l_l_thumb_ABD
- removed joint l_l_thumb_DIP
- removed joint l_l_thumb_MCP
- removed joint l_l_thumb_PIP
- removed joint l_l_wrist_FLEX
- removed joint l_l_wrist_PRO
- removed joint l_l_wrist_UDEV
- removed joint l_r_arm
- removed joint l_r_arm_twist
- removed joint pomocny1
- removed joint pomocny2
- removed joint r_arm
- removed joint r_arm_twist
- removed joint r_elbow
- removed joint r_elbow_twist
- added joint l_ankle_joint: type fixed, parent left_shin, child left_foot, origin xyz=0 -0.05 -0.44 rpy=0 0 0
- added joint l_arm_roll: type fixed, parent l_shoulder_lift, child l_upper_arm, origin xyz=0 0 0 rpy=0 0 0
- added joint l_elbow_flex: type fixed, parent l_upper_arm, child l_elbow_base, origin xyz=0 0 -0.23 rpy=0 0 0
- added joint l_elbow_roll: type fixed, parent l_elbow_base, child l_forearm, origin xyz=0 0 0 rpy=0 0 0
- added joint l_hip_joint: type fixed, parent pelvis, child left_thigh, origin xyz=0.09 -0.02 -0.065 rpy=0 0 0
- added joint l_index_ABD: type fixed, parent l_palm, child l_index0, origin xyz=-0.01 -0.066 0.001 rpy=0 -0.175 0
- added joint l_index_DIP: type fixed, parent l_index2, child l_index3, origin xyz=0.001 -0.025 0 rpy=0 0 0
- added joint l_index_MCP: type fixed, parent l_index0, child l_index1, origin xyz=0 -0.018 0 rpy=0 0 0
- added joint l_index_PIP: type fixed, parent l_index1, child l_index2, origin xyz=-0.001 -0.044 0.0005 rpy=0 0 0
- added joint l_knee_joint: type fixed, parent left_thigh, child left_shin, origin xyz=0 -0.01 -0.463 rpy=0 0 0
- added joint l_palm_joint: type fixed, parent l_wristz, child l_palm, origin xyz=-0.026 0 0 rpy=0 0 0
- added joint l_shoulder_lift: type fixed, parent l_shoulder_base, child l_shoulder_lift, origin xyz=0 0 0.12 rpy=0 0 0
- added joint l_shoulder_pan: type fixed, parent torso, child l_shoulder_base, origin xyz=0.20 -0.01 -0.06 rpy=0 0 0
- added joint l_wrist_FLEX: type fixed, parent l_wristx, child l_wristz, origin xyz=-0.0002 -0.03 -0.002 rpy=0 0 0
- added joint l_wrist_PRO: type fixed, parent l_forearm, child l_wristy, origin xyz=0 -0.23 0 rpy=0 0 0
- added joint l_wrist_UDEV: type fixed, parent l_wristy, child l_wristx, origin xyz=0 -0.048 0.002 rpy=0 0 0
- added joint lwaist_to_pelvis: type fixed, parent lwaist, child pelvis, origin xyz=0.0152 0 -0.185 rpy=0 -0.004 0
- added joint r_ankle_joint: type fixed, parent right_shin, child right_foot, origin xyz=0 -0.075 -0.44 rpy=0 0 0
- added joint r_arm_roll: type revolute, parent r_shoulder_lift, child r_upper_arm, origin xyz=0 0 0 rpy=0 0 0, axis 0 0 1, limit lower=-3.14 upper=3.14 effort=50 velocity=2.0
- added joint r_elbow_flex: type revolute, parent r_upper_arm, child r_elbow_base, origin xyz=0 0 -0.23 rpy=0 0 0, axis 1 0 0, limit lower=-2.8 upper=2.8 effort=50 velocity=2.0
- added joint r_elbow_roll: type revolute, parent r_elbow_base, child r_forearm, origin xyz=0 0 0 rpy=0 0 0, axis 0 0 1, limit lower=-3.14 upper=3.14 effort=30 velocity=2.0
- added joint r_hip_joint: type fixed, parent pelvis, child right_thigh, origin xyz=-0.12 -0.028 -0.065 rpy=0 0 0
- added joint r_knee_joint: type fixed, parent right_thigh, child right_shin, origin xyz=0 0.01 -0.463 rpy=0 0 0
- added joint r_palm_joint: type fixed, parent r_wristz, child r_palm, origin xyz=0.026 0 0 rpy=0 0 0
- added joint r_shoulder_lift: type revolute, parent r_shoulder_base, child r_shoulder_lift, origin xyz=0 0 0.12 rpy=0 0 0, axis 0 1 0, limit lower=-2.0 upper=1.57 effort=50 velocity=2.0
- added joint r_shoulder_pan: type revolute, parent torso, child r_shoulder_base, origin xyz=-0.20 -0.02 -0.06 rpy=0 0 0, axis 1 0 0, limit lower=-1.57 upper=2.0 effort=50 velocity=2.0
- added joint torso_to_head: type fixed, parent torso, child head, origin xyz=0 0 0.21 rpy=0 0 0
- added joint torso_to_lwaist: type fixed, parent torso, child lwaist, origin xyz=-0.01 0 -0.31 rpy=0 -0.004 0
- joint ee_x_axis_joint: origin xyz=0.0 0.0 0.1 rpy=0 0 0 -> xyz=0 -0.025 0 rpy=0 0 0
- joint ee_y_axis_joint: origin xyz=0.0 0.0 0.1 rpy=0 0 0 -> xyz=0 -0.025 0 rpy=0 0 0
- joint ee_z_axis_joint: origin xyz=0.0 0.0 0.1 rpy=0 0 0 -> xyz=0 -0.025 0 rpy=0 0 0
- joint endeffector_joint: origin xyz=0.0 0.0 0.1 rpy=0 3.14 0 -> xyz=0 -0.025 0 rpy=0 0 -1.5708
- joint joint_direction_cone: axis 0.00000 0.00000 0.00000 -> (none); origin xyz=0.00000 0.00000 0.00000 rpy=0.00000 -0.00000 0.00000 -> xyz=0 -0.025 0 rpy=0 0 0
- joint r_index_ABD: axis 0.00000 0.00000 1.00000 -> (none); child link0_23 -> r_index0; origin xyz=0.00986 -0.06580 0.00101 rpy=-0.00000 0.17453 -0.00000 -> xyz=0.01 -0.066 0.001 rpy=0 0.175 0
- joint r_index_DIP: axis 1.00000 0.00000 0.00000 -> (none); child link0_29 -> gripper; origin xyz=-0.00063 -0.02450 -0.00000 rpy=-0.00000 -0.00000 -0.00000 -> xyz=-0.001 -0.025 0 rpy=0 0 0
- joint r_index_MCP: axis 1.00000 0.00000 0.00000 -> (none); child link0_25 -> r_index1; origin xyz=0.00006 -0.01800 -0.00000 rpy=-0.00000 -0.00000 0.00000 -> xyz=0 -0.018 0 rpy=0 0 0
- joint r_index_PIP: axis 1.00000 0.00000 0.00000 -> (none); child link0_27 -> r_index2; origin xyz=0.00109 -0.04350 0.00050 rpy=0.00000 0.00000 0.00000 -> xyz=0.001 -0.044 0.0005 rpy=0 0 0
- joint r_wrist_FLEX: axis 1.00000 0.00000 0.00000 -> 1 0 0; child link0_12 -> r_wristz; limit (none) -> lower=-2.0 upper=2.0 effort=20 velocity=2.0; origin xyz=0.00019 -0.03000 -0.00209 rpy=0.00000 -0.00000 0.00000 -> xyz=0.0002 -0.03 -0.002 rpy=0 0 0; type continuous -> revolute
- joint r_wrist_PRO: axis 0.00000 1.00000 0.00000 -> 0 1 0; child link0_8 -> r_wristy; limit (none) -> lower=-3.14 upper=3.14 effort=20 velocity=2.0; origin xyz=-7.08369e-005 -0.0217787 -0.000286168 rpy=0.00000 -0.00000 0.00000 -> xyz=0 -0.23 0 rpy=0 0 0; type fixed -> revolute
- joint r_wrist_UDEV: axis 0.00000 0.00000 -1.00000 -> 0 0 -1; child link0_10 -> r_wristx; limit (none) -> lower=-1.57 upper=1.57 effort=20 velocity=2.0; origin xyz=-0.00003 -0.04765 0.00204 rpy=-0.00000 -0.00000 -0.00000 -> xyz=0 -0.048 0.002 rpy=0 0 0; type fixed -> revolute
